Commit message: 1/15 Updates

File: src/ripc_description/dynamics/ripc_dynamics_plugin.xacro (robot description, xacro)
@@ -5,5 +5,5 @@
       <!-- ================= BUOYANCY (MONOHULL) ================= -->
       <plugin filename="libSurface.so" name="vrx::Surface">
-        <!-- Apply buoyancy to hull -->
+        <!-- Apply buoyancy to base_link -->
         <link_name>base_link</link_name>
         <!-- Hull geometry -->
@@ -12,5 +12,5 @@
         <!-- Water surface height -->
         <fluid_level>0.0</fluid_level>
-        <!-- Buoyancy points along keel -->
+        <!-- Buoyancy points along keel needs to be symmetric about x-axis to prevent instability -->
         <points>
             <!-- Bow -->

File: src/ripc_description/dynamics/thruster_dynamics.xacro (robot description, xacro)
@@ -10,17 +10,17 @@
     <link name="${name}_propeller_link">
       <inertial>
-        <mass value="0.1"/>
-        <inertia ixx="0.0001" ixy="0.0" ixz="0.0"
-                 iyy="0.0001" iyz="0.0"
-                 izz="0.0001"/>
+        <mass value="0.3"/>
+        <inertia ixx="0.0003" ixy="0.0" ixz="0.0"
+                 iyy="0.0002" iyz="0.0"
+                 izz="0.0002"/>
       </inertial>
       <!-- Optional visual for debugging -->
       <visual>
-        <origin xyz="0 0 0" rpy="0 1.5708 0"/>
+        <origin xyz="0 0 0" rpy="0 0 -1.5708"/>
         <geometry>
-          <cylinder radius="0.05" length="0.01"/>
+          <mesh filename="package://ripc_description/meshes/prop.dae" scale="1 1 1"/>
         </geometry>
         <material name="propeller_gray">
-          <color rgba="0.3 0.3 0.3 1.0"/>
+          <color rgba="1.0 0.0 0.0 1.0"/>
         </material>
       </visual>
@@ -40,5 +40,5 @@
         <thrust_coefficient>0.004422</thrust_coefficient>
         <fluid_density>1000</fluid_density>
-        <propeller_diameter>0.1</propeller_diameter>
+        <propeller_diameter>0.191</propeller_diameter>
         <velocity_control>true</velocity_control>
         <max_thrust_cmd>80</max_thrust_cmd>
@@ -56,10 +56,10 @@
                          name="left"
                          parent_link="${parent_link}"
-                         xyz="-0.5192 0.1778 -0.1905"/>
+                         xyz="-0.5462 0.1778 -0.1905"/>
     <!-- Right thruster -->
     <xacro:ripc_thruster namespace="${namespace}"
                          name="right"
                          parent_link="${parent_link}"
-                         xyz="-0.5192 -0.1778 -0.1905"/>
+                         xyz="-0.5462 -0.1778 -0.1905"/>
   </xacro:macro>
 </robot>

File: src/ripc_description/urdf/ripc_usv.urdf.xacro (robot description, xacro)
@@ -1,4 +1,7 @@
 <?xml version="1.0"?>
 <robot xmlns:xacro="http://ros.org/wiki/xacro" name="ripc_usv">
+  <!--Include sensor links and physical properties-->
+  <xacro:include filename="$(find ripc_gazebo)/sensors/imu.xacro"/>
+  <xacro:sensors namespace="ripc_usv" parent_link="base_link" xyz="0.5 0 0.2" rpy="0 0 0" />
   <!-- Include dynamics plugin macros -->
   <xacro:include filename="$(find ripc_description)/dynamics/ripc_dynamics_plugin.xacro"/>
@@ -12,12 +15,14 @@
   </link>
   <!-- ================== Hull ================== -->
+  <!-- Assume non-zero diagnoal values because of the hull's shape and mass distribution -->
   <link name="hull">
     <inertial>
-      <origin xyz="0 0 0" rpy="0 0 0"/>
-      <mass value="120"/>
-      <inertia ixx="120" ixy="0.0" ixz="0.0"
-               iyy="393" iyz="0.0"
-               izz="446"/>
+      <origin xyz="0 0 -0.15" rpy="0 0 0"/>
+      <mass value="131"/>
+      <inertia ixx="20" ixy="0.0" ixz="0.0"
+               iyy="42" iyz="0.0"
+               izz="42"/>
     </inertial>
+    <!--  -->
     <visual>
       <origin xyz="0.446 0 0.0127" rpy="0 0 1.5708"/>
@@ -26,16 +31,16 @@
       </geometry>
       <material name="ripc_hull_color">
-        <color rgba="0.1 0.2 0.8 1.0"/>
+        <color rgba="0.0 1.0 0.0 1.0"/>
       </material>
     </visual>
-      <!-- SIMPLE collision box -->
+    <!-- SIMPLE collision box -->
     <collision name="hull_collision_box">
-      <origin xyz="0 0 -0.106" rpy="0 0 0"/>
+      <origin xyz="0.125 0 0.05" rpy="0 0 0"/>
       <geometry>
-        <box size="1.45 0.70 0.20"/>
+        <box size="1.54 0.725 0.67"/>
       </geometry>
     </collision>
   </link>
-  <!-- Fixed joint from base_link to hull -->
+  <!-- Fixed joint from base_link to hull, makes it so base_link and hull have same frame and essentially behave as one -->
   <joint name="base_to_hull" type="fixed">
     <parent link="base_link"/>

File: src/ripc_gazebo/plugins/ripc_plugins.xacro (robot description, xacro)
@@ -16,4 +16,13 @@
       <preserveFixedJoint>true</preserveFixedJoint>
     </gazebo>
+    <gazebo>
+      <plugin
+        filename="gz-sim-joint-state-publisher-system"
+        name="gz::sim::systems::JointStatePublisher">
+        <joint_name>ripc_usv_left_propellor_joint</joint_name>
+        <joint_name>ripc_usv_right_propellor_joint</joint_name>
+        <topic>/model/ripc_usv/joint_states</topic>
+      </plugin>
+    </gazebo>
   </xacro:macro>
 </robot>
