Commit message: 1/18 Updae

File: src/ripc_description/dynamics/thruster_dynamics.xacro (robot description, xacro)
@@ -63,3 +63,9 @@
                          xyz="-0.5462 -0.1778 -0.1905"/>
   </xacro:macro>
+  <gazebo reference="ripc_usv_left_propeller_joint">
+    <preserveFixedJoint>true</preserveFixedJoint>
+  </gazebo>
+  <gazebo reference="ripc_usv_right_propeller_joint">
+    <preserveFixedJoint>true</preserveFixedJoint>
+  </gazebo>
 </robot>

File: src/ripc_description/urdf/ripc_usv.urdf.xacro (robot description, xacro)
@@ -3,5 +3,8 @@
   <!--Include sensor links and physical properties-->
   <xacro:include filename="$(find ripc_gazebo)/sensors/imu.xacro"/>
-  <xacro:sensors namespace="ripc_usv" parent_link="base_link" xyz="0.5 0 0.2" rpy="0 0 0" />
+  <xacro:imu_sensor_macro namespace="ripc_usv" parent_link="base_link" imu_name="imu_bow" xyz="0.77 0 0.5" rpy="0 0 0" />
+  <xacro:imu_sensor_macro namespace="ripc_usv" parent_link="base_link" imu_name="imu_stern" xyz="-0.77 0 0.5" rpy="0 0 0" />
+  <xacro:include filename="$(find ripc_gazebo)/sensors/gps.xacro" />
+  <xacro:gps_sensor name="gps" parent="base_link" x="0.0" y="0.0" z="1.5" />
   <!-- Include dynamics plugin macros -->
   <xacro:include filename="$(find ripc_description)/dynamics/ripc_dynamics_plugin.xacro"/>
@@ -42,5 +45,4 @@
     </collision>
   </link>
-  <!-- Fixed joint from base_link to hull, makes it so base_link and hull have same frame and essentially behave as one -->
   <joint name="base_to_hull" type="fixed">
     <parent link="base_link"/>

File: src/ripc_gazebo/plugins/ripc_plugins.xacro (robot description, xacro)
@@ -2,5 +2,5 @@
 <robot xmlns:xacro="http://ros.org/wiki/xacro">
   <xacro:macro name="ripc_plugins" params="namespace">
-    <gazebo>
+   <gazebo>
       <plugin
         filename="gz-sim-odometry-publisher-system"
@@ -10,4 +10,5 @@
         <odom_topic>/model/${namespace}/odometry</odom_topic>
         <tf_topic>/model/${namespace}/tf</tf_topic>
+        <publish_tf>false</publish_tf>
         <odom_publish_frequency>50</odom_publish_frequency>
       </plugin>
@@ -20,6 +21,9 @@
         filename="gz-sim-joint-state-publisher-system"
         name="gz::sim::systems::JointStatePublisher">
-        <joint_name>ripc_usv_left_propellor_joint</joint_name>
-        <joint_name>ripc_usv_right_propellor_joint</joint_name>
+        <update_rate>50</update_rate>
+        <joint_name>ripc_usv_left_propeller_joint</joint_name>
+        <joint_name>ripc_usv_right_propeller_joint</joint_name>
+        <joint_name>imu_bow_joint</joint_name>
+        <joint_name>imu_stern_joint</joint_name>
         <topic>/model/ripc_usv/joint_states</topic>
       </plugin>

File: src/ripc_gazebo/sensors/imu.xacro (robot description, xacro)
@@ -1,40 +1,44 @@
 <?xml version="1.0"?>
 <robot xmlns:xacro="http://ros.org/wiki/xacro">
-  <xacro:macro name="sensors" params="namespace parent_link xyz:='0 0 0' rpy:='0 0 0'">
-    <link name="imu_link">
+  <xacro:macro name="imu_sensor_macro" params="namespace parent_link imu_name xyz rpy">
+    <link name="${imu_name}_link">
       <inertial>
         <mass value="0.01"/>
-        <origin xyz="0 0 0" rpy="0 0 0"/>
         <inertia ixx="1e-7" ixy="0" ixz="0" iyy="1e-7" iyz="0" izz="1e-7"/>
       </inertial>
-      <visual>
+      <collision>
         <geometry>
-          <box size="0.05 0.05 0.02"/>
+            <box size="0.01 0.01 0.01"/>
         </geometry>
-      </visual>
+      </collision>
     </link>
-    <joint name="imu_joint" type="fixed">
-      <parent link="${parent_link}"/>
-      <child link="imu_link"/>
-      <origin xyz="${xyz}" rpy="${rpy}"/>
+    <joint name="${imu_name}_joint" type="revolute">
+        <parent link="${parent_link}"/>
+        <child link="${imu_name}_link"/>
+        <origin xyz="${xyz}" rpy="${rpy}"/>
+        <limit effort="0" lower="0" upper="0" velocity="0"/>
     </joint>
-    <gazebo reference="imu_joint">
+    <gazebo reference="${imu_name}_link">
+      <sensor name="${imu_name}" type="imu">
+        <always_on>1</always_on>
+        <update_rate>100</update_rate>
+        <topic>/model/${namespace}/${imu_name}</topic>
+        <gz_frame_id>${imu_name}_link</gz_frame_id>
+        <imu>
+          <angular_velocity>
+            <x><noise type="gaussian"><stddev>2e-4</stddev></noise></x>
+            <y><noise type="gaussian"><stddev>2e-4</stddev></noise></y>
+            <z><noise type="gaussian"><stddev>2e-4</stddev></noise></z>
+          </angular_velocity>
+          <linear_acceleration>
+            <x><noise type="gaussian"><stddev>1.7e-2</stddev></noise></x>
+            <y><noise type="gaussian"><stddev>1.7e-2</stddev></noise></y>
+            <z><noise type="gaussian"><stddev>1.7e-2</stddev></noise></z>
+          </linear_acceleration>
+        </imu>
+      </sensor>
+    </gazebo>
+    <gazebo reference="${imu_name}_joint">
       <preserveFixedJoint>true</preserveFixedJoint>
     </gazebo>
-    <gazebo reference="imu_link">
-      <sensor name="imu_sensor" type="imu">
-        <always_on>1</always_on>
-        <update_rate>100</update_rate>
-        <visualize>true</visualize>
-        <topic>/model/${namespace}/imu</topic>
-        <gz_frame_id>imu_link</gz_frame_id>
-      </sensor>
-    </gazebo>
-    <gazebo>
-      <plugin
-        filename="gz-sim-imu-system"
-        name="gz::sim::systems::Imu">
-      </plugin>
-    </gazebo>
-  </xacro:macro>
-</robot>
+  </xacro:macro> </robot>

Commit message: 2/22

File: src/ripc_description/dynamics/thruster_dynamics.xacro (robot description, xacro)
@@ -32,4 +32,5 @@
       <origin xyz="${xyz}" rpy="0 0 0"/>
       <axis xyz="1 0 0"/>
+      <dynamics friction="0.05" damping="0.05"/>
     </joint>
     <!-- Gazebo Thruster plugin -->

File: src/ripc_gazebo/plugins/ripc_plugins.xacro (robot description, xacro)
@@ -10,6 +10,7 @@
         <odom_topic>/model/${namespace}/odometry</odom_topic>
         <tf_topic>/model/${namespace}/tf</tf_topic>
-        <publish_tf>false</publish_tf>
+        <publish_tf>true</publish_tf>
         <odom_publish_frequency>50</odom_publish_frequency>
+        <dimensions>2</dimensions>
       </plugin>
     </gazebo>

Commit message: RVIZ2 With URDF

File: src/ripc_description/dynamics/thruster_dynamics.xacro (robot description, xacro)
@@ -27,5 +27,5 @@
     </link>
     <!-- Continuous joint for spinning -->
-    <joint name="${namespace}_${name}_propeller_joint" type="continuous">
+    <joint name="${namespace}_${name}_propeller_joint" type="fixed">
       <parent link="${parent_link}"/>
       <child link="${name}_propeller_link"/>

File: src/ripc_description/urdf/ripc_usv.urdf.xacro (robot description, xacro)
@@ -20,5 +20,5 @@
   <!-- ================== Hull ================== -->
   <!-- Assume non-zero diagnoal values because of the hull's shape and mass distribution -->
-  <link name="hull">
+  <!-- <link name="hull">
     <inertial>
       <origin xyz="0 0 -0.15" rpy="0 0 0"/>
@@ -27,5 +27,5 @@
                iyy="42" iyz="0.0"
                izz="42"/>
-    </inertial>
+    </inertial> -->
     <!--  -->
     <visual>
@@ -38,5 +38,5 @@
       </material>
     </visual>
-    <!-- SIMPLE collision box -->
+    <!-- SIMPLE collision box
     <collision name="hull_collision_box">
       <origin xyz="0.125 0 0.05" rpy="0 0 0"/>
@@ -44,10 +44,10 @@
         <box size="1.54 0.725 0.67"/>
       </geometry>
-    </collision>
-  </link>
-  <joint name="base_to_hull" type="fixed">
+    </collision> -->
+  <!-- </link> -->
+  <!-- <joint name="base_to_hull" type="fixed">
     <parent link="base_link"/>
     <child link="hull"/>
     <origin xyz="0 0 0" rpy="0 0 0"/>
-  </joint>
+  </joint> -->
 </robot>

File: src/ripc_gazebo/sensors/gps.xacro (robot description, xacro)
@@ -2,5 +2,5 @@
 <robot xmlns:xacro="http://www.ros.org/wiki/xacro">
   <xacro:macro name="gps_sensor" params="name parent x y z">
-    <joint name="${name}_joint" type="revolute">
+    <joint name="${name}_joint" type="fixed">
         <parent link="${parent}"/>
         <child link="${name}_link"/>

File: src/ripc_gazebo/sensors/imu.xacro (robot description, xacro)
@@ -13,5 +13,5 @@
       </collision>
     </link>
-    <joint name="${imu_name}_joint" type="revolute">
+    <joint name="${imu_name}_joint" type="fixed">
         <parent link="${parent_link}"/>
         <child link="${imu_name}_link"/>
