Commit message: 1/2/26 Updates

File: src/ripc_description/urdf/ripc_usv.urdf.xacro (robot description, xacro)
@@ -1,7 +1,11 @@
 <?xml version="1.0"?>
 <robot xmlns:xacro="http://ros.org/wiki/xacro" name="ripc_usv">
+  <!-- Include dynamics plugin macros -->
+  <xacro:include filename="$(find ripc_description)/dynamics/ripc_dynamics_plugin.xacro"/>
+  <xacro:include filename="$(find ripc_description)/dynamics/thruster_dynamics.xacro"/>
+    <xacro:ripc_thrusters namespace="ripc_usv" parent_link="base_link"/>
+  <xacro:usv_dynamics_gazebo namespace="ripc_usv"/>
   <!-- ================== Base link / Dummy root ================== -->
   <link name="base_link">
-    <!-- Dummy root, no visual/collision -->
   </link>
   <!-- ================== Hull ================== -->
@@ -9,8 +13,8 @@
     <inertial>
       <origin xyz="0 0 0" rpy="0 0 0"/>
-      <mass value="50.0"/>
-      <inertia ixx="5.0" ixy="0.0" ixz="0.0"
-               iyy="5.0" iyz="0.0"
-               izz="10.0"/>
+      <mass value="120"/>
+      <inertia ixx="120" ixy="0.0" ixz="0.0"
+               iyy="393" iyz="0.0"
+               izz="446"/>
     </inertial>
     <visual>
@@ -23,8 +27,9 @@
       </material>
     </visual>
-    <collision>
-      <origin xyz="0.446 0 0.0127" rpy="0 0 1.5708"/>
+      <!-- SIMPLE collision box -->
+    <collision name="hull_collision_box">
+      <origin xyz="0 0 -0.106" rpy="0 0 0"/>
       <geometry>
-        <mesh filename="package://ripc_description/meshes/ripc_usv.dae" scale="1 1 1"/>
+        <box size="1.45 0.70 0.20"/>
       </geometry>
     </collision>
@@ -36,31 +41,3 @@
     <origin xyz="0 0 0" rpy="0 0 0"/>
   </joint>
-  <!-- ================== Left Propeller ================== -->
-  <link name="left_propeller_link">
-    <inertial>
-      <mass value="0.1"/>
-      <inertia ixx="0.0001" ixy="0.0" ixz="0.0" iyy="0.0001" iyz="0.0" izz="0.0001"/>
-    </inertial>
-    <!-- Visual removed, can add mesh later -->
-  </link>
-  <joint name="left_propeller_joint" type="continuous">
-    <parent link="hull"/>
-    <child link="left_propeller_link"/>
-    <origin xyz="-0.5192 0.1778 -0.1905" rpy="0 0 0"/>
-    <axis xyz="1 0 0"/>
-  </joint>
-  <!-- ================== Right Propeller ================== -->
-  <link name="right_propeller_link">
-    <inertial>
-      <mass value="0.1"/>
-      <inertia ixx="0.0001" ixy="0.0" ixz="0.0" iyy="0.0001" iyz="0.0" izz="0.0001"/>
-    </inertial>
-    <!-- Visual removed, can add mesh later -->
-  </link>
-  <joint name="right_propeller_joint" type="continuous">
-    <parent link="hull"/>
-    <child link="right_propeller_link"/>
-    <origin xyz="-0.5192 -0.1778 -0.1905" rpy="0 0 0"/>
-    <axis xyz="1 0 0"/>
-  </joint>
 </robot>

Commit message: 1/19 Update

File: src/ripc_description/urdf/ripc_usv.urdf.xacro (robot description, xacro)
@@ -6,5 +6,5 @@
   <xacro:imu_sensor_macro namespace="ripc_usv" parent_link="base_link" imu_name="imu_stern" xyz="-0.77 0 0.5" rpy="0 0 0" />
   <xacro:include filename="$(find ripc_gazebo)/sensors/gps.xacro" />
-  <xacro:gps_sensor name="gps" parent="base_link" x="0.0" y="0.0" z="1.5" />
+  <xacro:gps_sensor name="gps" parent="base_link" x="0.0" y="0.0" z="0.75" />
   <!-- Include dynamics plugin macros -->
   <xacro:include filename="$(find ripc_description)/dynamics/ripc_dynamics_plugin.xacro"/>

File: src/ripc_gazebo/sensors/gps.xacro (robot description, xacro)
@@ -2,8 +2,10 @@
 <robot xmlns:xacro="http://www.ros.org/wiki/xacro">
   <xacro:macro name="gps_sensor" params="name parent x y z">
-    <joint name="${name}_joint" type="fixed">
-      <parent link="${parent}"/>
-      <child link="${name}_link"/>
-      <origin xyz="${x} ${y} ${z}" rpy="0 0 0"/>
+    <joint name="gps_joint" type="revolute">
+        <parent link="base_link"/>
+        <child link="gps_link"/>
+        <origin xyz="0.0 0.0 0.75" rpy="0 0 0"/>
+        <axis xyz="0 0 1"/>
+        <limit lower="0" upper="0" effort="0" velocity="0"/>
     </joint>
     <link name="${name}_link">
