Commit message: 1/21 Updates

File: src/ripc_gazebo/plugins/ripc_plugins.xacro (robot description, xacro)
@@ -26,4 +26,5 @@
         <joint_name>imu_bow_joint</joint_name>
         <joint_name>imu_stern_joint</joint_name>
+        <joint_name>gps_joint</joint_name>
         <topic>/model/ripc_usv/joint_states</topic>
       </plugin>

File: src/ripc_gazebo/sensors/gps.xacro (robot description, xacro)
@@ -7,5 +7,5 @@
         <origin xyz="0.0 0.0 0.75" rpy="0 0 0"/>
         <axis xyz="0 0 1"/>
-        <limit lower="0" upper="0" effort="0" velocity="0"/>
+        <limit lower="0.0" upper="0.0" effort="0" velocity="0"/>
     </joint>
     <link name="${name}_link">
@@ -31,4 +31,7 @@
       </sensor>
     </gazebo>
+    <gazebo reference="gps_joint">
+      <preserveFixedJoint>true</preserveFixedJoint>
+    </gazebo>
   </xacro:macro>
 </robot>
